File: pcb/car.sch (KiCad schematic (older format))
At the start: 22 parts, among them J1 LED strip front, J2 12V fused out, J3 Car power, Q1 2N222A, Q2 2N222A, Q3 2N222A, Q4 2N3906, U1 LM7805, U2 5v-relais

Commit message: Draft schematic: Arduino Nano, MCP2515 CAN module and 12V power latch
Parts:
- removed J1: LED strip front, symbol Screw_Terminal_01x03
- removed Q1, Q2, Q3: 2N222A, TO_SOT_Packages_THT:TO-39-3, symbol 2N2219
- removed R1, R2, R3: R, symbol R
- added C4: 1uF, symbol car-rescue:CP1_Small
- added D3, D4: 1N4148, symbol car-rescue:D
- added F2: Fuse, symbol car-rescue:Fuse
- added Q1, Q5, Q7: 2N3904, Package_TO_SOT_THT:TO-92_Inline, symbol Transistor_BJT:2N3904
- added Q2: IRF4905, Package_TO_SOT_THT:TO-220-3_Vertical, symbol Transistor_FET:IRF4905
- added Q3, Q6: NDP6020P, Package_TO_SOT_THT:TO-220-3_Vertical, symbol Transistor_FET:IRF4905
- added R1: 100K, symbol car-rescue:R
- added R10, R11, R3, R7, R8, R9, R?: 10K, symbol Device:R
- added U3: LM7805, TO_SOT_Packages_THT:TO-220_Vertical, symbol car-rescue:LM7805_TO220
- added XA2: Arduino_Nano_Socket, symbol arduino:Arduino_Nano_Socket
- C1: symbol CP -> car-rescue:CP
- C2, C3: symbol CP1_Small -> car-rescue:CP1_Small
- D1, D2: symbol D -> car-rescue:D
- F1: symbol Fuse -> car-rescue:Fuse
- J2, J3: symbol Screw_Terminal_01x03 -> car-rescue:Screw_Terminal_01x03
- Q4: symbol 2N3906 -> car-rescue:2N3906
- R4, R5, R6: symbol R -> car-rescue:R
- U1: symbol LM7805_TO220 -> car-rescue:LM7805_TO220
- U2: symbol 5v-relais -> arduino:5v-relais
- XA1: symbol Arduino_Nano_Socket -> arduino:Arduino_Nano_Socket
Connections:
- net labels added: +5V, 12V_MAIN, 12V_Switched, Can, NEOLEFT, NEORIGHT, OUTPUT_1, OUTPUT_2
- wire segments 57 -> 78
Other:
- note added: "Dc-DC converter 5v\n"
- note added: "MCP2512 Can Module\n"
- moved on the sheet: C1, C2, C3, D1, D2, F1, J2, J3, Q4, R4, R5, R6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
